Commit message: Add dummy links for SITL control

File: bluerov2_description/urdf/actuators.xacro (robot description, xacro)
@@ -37,3 +37,49 @@
     <origin xyz="0 0 0" rpy="0 0 0"/>
   </xacro:default_beacon> -->
+  <!-- ### -->
+  <!-- IMPROVE -->
+  <!-- Add dummy links & joints for ArduPilotPlugin -->
+  <!-- From uuv-simulator -->
+  <xacro:macro name="ap_dummy_thruster_macro" params="robot_namespace thruster_id *origin">
+    <!--
+    Dummy link for ArduPilot to attach to
+    -->
+    <link name="${robot_namespace}/ap_dummy_thruster_${thruster_id}">
+      <inertial>
+        <mass value="0.010" />
+        <origin xyz="0 0 0" rpy="0 0 0"/>
+        <inertia ixx="0.00001" ixy="0.0" ixz="0.0"
+               iyy="0.00001" iyz="0.0"
+               izz="0.00001" />
+      </inertial>
+    </link>
+    <joint name="${robot_namespace}/ap_dummy_thruster_${thruster_id}_joint" type="revolute">
+      <xacro:insert_block name="origin" />
+      <axis xyz="1 0 0" />
+      <limit effort="0.0" upper="0.0" lower="0.0" velocity="0.0"/>
+      <parent link="${robot_namespace}/base_link" />
+      <child link="${robot_namespace}/ap_dummy_thruster_${thruster_id}" />
+    </joint>
+    <gazebo reference="${robot_namespace}/ap_dummy_thruster_${thruster_id}">
+      <selfCollide>false</selfCollide>
+    </gazebo>
+  </xacro:macro>
+  <xacro:ap_dummy_thruster_macro robot_namespace="${namespace}" thruster_id="0">
+    <origin xyz="0.1355 -0.1 -0.0725" rpy="1.5707963 1.5707963 -0.78539815"/>
+  </xacro:ap_dummy_thruster_macro>
+  <xacro:ap_dummy_thruster_macro robot_namespace="${namespace}" thruster_id="1">
+    <origin xyz="0.1355 0.1 -0.0725" rpy="1.5707963 1.5707963 3.92699075"/>
+  </xacro:ap_dummy_thruster_macro>
+  <xacro:ap_dummy_thruster_macro robot_namespace="${namespace}" thruster_id="2">
+    <origin xyz="-0.1475 -0.1 -0.0725" rpy="1.5707963 1.5707963 0.78540075"/>
+  </xacro:ap_dummy_thruster_macro>
+  <xacro:ap_dummy_thruster_macro robot_namespace="${namespace}" thruster_id="3">
+    <origin xyz="-0.1475 0.1 -0.0725" rpy="1.5707963 1.5707963 2.35619445"/>
+  </xacro:ap_dummy_thruster_macro>
+  <xacro:ap_dummy_thruster_macro robot_namespace="${namespace}" thruster_id="4">
+    <origin xyz="0.0025 -0.1105 -0.005" rpy="3.1415926 0 0"/>
+  </xacro:ap_dummy_thruster_macro>
+  <xacro:ap_dummy_thruster_macro robot_namespace="${namespace}" thruster_id="5">
+    <origin xyz="0.0025 0.1105 -0.005" rpy="3.1415926 0 0"/>
+  </xacro:ap_dummy_thruster_macro>
 </robot>
