Commit message: Add Realsense camera in sensors.xacro

File: bluerov2_description/urdf/sensors.xacro (robot description, xacro)
@@ -26,3 +26,15 @@
   <!-- Mount a GPS. -->
   <xacro:default_gps namespace="${namespace}" parent_link="${namespace}/base_link" />
+  <!-- ### -->
+  <!-- Add RealSense camera support -->
+  <xacro:include filename="$(find realsense2_description)/urdf/_d435.urdf.xacro" />
+  <xacro:sensor_d435 parent="${namespace}/base_link"
+    use_nominal_extrinsics="true"
+    add_plug="false"
+    use_mesh="true"
+    name="camera"
+    topics_ns="camera"
+    publish_pointcloud="true">
+    <origin xyz="0.2 0 0" rpy="0 0 0"/>
+  </xacro:sensor_d435>
 </robot>

Commit message: Fixed down camera - topic /bluerov2/camera_down/camera_image

File: bluerov2_description/urdf/sensors.xacro (robot description, xacro)
@@ -17,11 +17,19 @@
     <origin xyz="0 0 0" rpy="0 0 0"/>
   </xacro:default_pressure>
+  <!-- Sonar Sensor -->
+  <!-- <xacro:bluerov_altimeter namespace="${namespace}" parent_link="${namespace}/base_link">
+    <origin xyz="0 0 -0.2" rpy="0 ${pi/2} 0"/>
+  </xacro:bluerov_altimeter> -->
   <!-- Mount a camera -->
-  <xacro:bluerov_camera namespace="" parent_link="${namespace}/base_link" suffix="_front">
+  <xacro:bluerov_camera namespace="" parent_link="${namespace}/base_link" suffix="_down"
+    width="640" height="400" hfov="1.2">
+    <origin xyz="0 0 -0.14" rpy="0 ${pi/2} 0"/>
+  </xacro:bluerov_camera>
+  <!-- <xacro:bluerov_camera namespace="" parent_link="${namespace}/base_link" suffix="_front">
     <origin xyz="0.2 0 0" rpy="0 0 0"/>
-  </xacro:bluerov_camera>
-  <xacro:bluerov_camera namespace="" parent_link="${namespace}/base_link" suffix="_down">
-    <origin xyz="0 0 -0.2" rpy="0 ${pi/2} 0"/>
-  </xacro:bluerov_camera>
+  </xacro:bluerov_camera> -->
+  <!-- <xacro:bluerov_camera namespace="" parent_link="${namespace}/base_link" suffix="_down">
+    <origin xyz="0 0 -0.11" rpy="0 ${pi/2} 0"/>
+  </xacro:bluerov_camera> -->
   <!-- Mount a GPS. -->
   <xacro:default_gps namespace="${namespace}" parent_link="${namespace}/base_link" />

File: bluerov2_description/urdf/snippets.xacro (robot description, xacro)
@@ -84,5 +84,5 @@
     </gazebo>
   </xacro:macro>
-  <xacro:macro name="bluerov_camera" params="namespace parent_link suffix *origin">
+  <xacro:macro name="bluerov_camera" params="namespace parent_link suffix width height hfov *origin">
     <xacro:regular_camera_plugin_macro
       namespace="${namespace}"
@@ -92,7 +92,7 @@
       mass="0.001"
       update_rate="30"
-      hfov="1.5125"
-      width="1920"
-      height="1080"
+      hfov="${hfov}"
+      width="${width}"
+      height="${height}"
       stddev="0.01"
       scale="1.0">
